File: hardware/io_board.brd (EAGLE design)
At the start: 151.4 x 117.5 mm, 54 parts, among them IC1 74HC76N, IC2 MAX232, IC3 74HC76N, IC5 7486N, IC6 74HCT138N, IC7 7486N, IC8 74HCT04N, X3 22-23-2051, X4 22-23-2051, X5 22-23-2021

Commit message: IO board modified
Connections:
- net N$1 renamed TXD_TTL
- net N$3 renamed RXD_TTL
- removed net N$2: IC2.10, U1.8
- removed net N$4: IC2.9, U1.9
- net GND: now also U1.9
Routing:
- net N$2: track 35.0 -> 0.00 mm, vias 2 -> 0
- net N$4: track 33.7 -> 0.00 mm, vias 2 -> 0
- net GND: track 127.3 -> 147.1 mm, vias 21 -> 23
Changed lines of the file:
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@@
 <?xml version="1.0" encoding="utf-8"?>
 <!DOCTYPE eagle SYSTEM "eagle.dtd">
-<eagle version="7.2.0">
+<eagle version="7.7.0">
 <drawing>
 <settings>
@@
 <contactref element="C20" pad="-"/>
 <contactref element="C21" pad="2"/>
-<wire x1="118.745" y1="36.7" x2="118.745" y2="39.5" width="0" layer="19" extent="16-16"/>
+<contactref element="U1" pad="9"/>
+<wire x1="126.6825" y1="60.325" x2="125.095" y2="60.325" width="0.4064" layer="16"/>
+<wire x1="125.095" y1="60.325" x2="123.825" y2="59.055" width="0.4064" layer="16"/>
+<wire x1="123.825" y1="59.055" x2="118.11" y2="59.055" width="0.4064" layer="16"/>
+<via x="118.11" y="59.055" extent="1-16" drill="0.6" diameter="1.4224" shape="octagon"/>
+<wire x1="118.11" y1="59.055" x2="118.11" y2="69.85" width="0.4064" layer="1"/>
+<via x="118.11" y="69.85" extent="1-16" drill="0.6" diameter="1.4224" shape="octagon"/>
+<wire x1="118.745" y1="39.5" x2="118.745" y2="36.7" width="0" layer="19" extent="16-16"/>
 </signal>
 <signal name="D0">
@@
 <via x="145.97" y="112.315" extent="1-16" drill="0.6" diameter="1.9304"/>
 </signal>
-<signal name="N$1">
+<signal name="TXD_TTL">
 <contactref element="U1" pad="10"/>
 <contactref element="IC2" pad="11"/>
@@
 <wire x1="121.6025" y1="78.105" x2="119.38" y2="75.8825" width="0.4064" layer="16"/>
 </signal>
-<signal name="N$2">
-<contactref element="U1" pad="8"/>
-<contactref element="IC2" pad="10"/>
-<wire x1="126.6825" y1="57.785" x2="125.095" y2="57.785" width="0.4064" layer="16"/>
-<wire x1="125.095" y1="57.785" x2="123.825" y2="56.515" width="0.4064" layer="16"/>
-<wire x1="123.825" y1="56.515" x2="120.65" y2="56.515" width="0.4064" layer="16"/>
-<via x="120.65" y="56.515" extent="1-16" drill="0.6" diameter="1.4224" shape="octagon"/>
-<wire x1="120.65" y1="56.515" x2="120.65" y2="80.645" width="0.4064" layer="1"/>
-<via x="120.65" y="80.645" extent="1-16" drill="0.6" diameter="1.4224" shape="octagon"/>
-<wire x1="124.1425" y1="82.55" x2="122.555" y2="82.55" width="0.6096" layer="16"/>
-<wire x1="122.555" y1="82.55" x2="120.65" y2="80.645" width="0.6096" layer="16"/>
-</signal>
-<signal name="N$3">
+<signal name="RXD_TTL">
 <contactref element="U1" pad="12"/>
 <contactref element="IC2" pad="12"/>
@@
 <wire x1="126.365" y1="87.63" x2="124.1425" y2="87.63" width="0.4064" layer="16"/>
 </signal>
-<signal name="N$4">
-<contactref element="U1" pad="9"/>
-<contactref element="IC2" pad="9"/>
-<wire x1="126.6825" y1="60.325" x2="125.095" y2="60.325" width="0.4064" layer="16"/>
-<wire x1="125.095" y1="60.325" x2="123.825" y2="59.055" width="0.4064" layer="16"/>
-<wire x1="123.825" y1="59.055" x2="118.11" y2="59.055" width="0.4064" layer="16"/>
-<via x="118.11" y="59.055" extent="1-16" drill="0.6" diameter="1.4224" shape="octagon"/>
-<wire x1="118.11" y1="59.055" x2="118.11" y2="75.8825" width="0.4064" layer="1"/>
-<via x="118.11" y="75.8825" extent="1-16" drill="0.6" diameter="1.4224" shape="octagon"/>
-<wire x1="124.1425" y1="80.01" x2="122.2375" y2="80.01" width="0.4064" layer="16"/>
-<wire x1="122.2375" y1="80.01" x2="118.11" y2="75.8825" width="0.4064" layer="16"/>
-</signal>
 <signal name="N$5">
