File: hardware/io_board.sch (EAGLE design)
At the start: 54 parts, among them IC1 74HC76N, IC2 MAX232, IC3 74HC76N, IC5 7486N, IC6 74HCT138N, IC7 7486N, IC8 74HCT04N, X3 22-23-2051, X4 22-23-2051, X5 22-23-2021

Commit message: IO board modified
Connections:
- net N$1 renamed TXD_TTL
- net N$3 renamed RXD_TTL
- removed net N$2: IC2G$1.T2IN, U1.RTS
- removed net N$4: IC2G$1.R2OUT, U1.CTS
- net GND: now also U1.CTS
Changed lines of the file:
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@@
 <?xml version="1.0" encoding="utf-8"?>
 <!DOCTYPE eagle SYSTEM "eagle.dtd">
-<eagle version="7.2.0">
+<eagle version="7.7.0">
 <drawing>
 <settings>
@@
 <wire x1="5.08" y1="55.88" x2="7.62" y2="55.88" width="0.1524" layer="91"/>
 <junction x="7.62" y="55.88"/>
+<pinref part="U1" gate="G$1" pin="CTS"/>
+<wire x1="5.08" y1="60.96" x2="7.62" y2="60.96" width="0.1524" layer="91"/>
+<wire x1="7.62" y1="60.96" x2="7.62" y2="58.42" width="0.1524" layer="91"/>
+<junction x="7.62" y="58.42"/>
 </segment>
 <segment>
@@
 </segment>
 </net>
-<net name="N$1" class="0">
+<net name="TXD_TTL" class="0">
 <segment>
 <pinref part="U1" gate="G$1" pin="TXD"/>
@@
 </segment>
 </net>
-<net name="N$2" class="0">
-<segment>
-<pinref part="U1" gate="G$1" pin="RTS"/>
-<wire x1="5.08" y1="48.26" x2="38.1" y2="48.26" width="0.1524" layer="91"/>
-<pinref part="IC2" gate="G$1" pin="T2IN"/>
-</segment>
-</net>
-<net name="N$3" class="0">
+<net name="RXD_TTL" class="0">
 <segment>
 <pinref part="U1" gate="G$1" pin="RXD"/>
@@
 </segment>
 </net>
-<net name="N$4" class="0">
-<segment>
-<pinref part="U1" gate="G$1" pin="CTS"/>
-<wire x1="5.08" y1="60.96" x2="17.78" y2="60.96" width="0.1524" layer="91"/>
-<wire x1="17.78" y1="60.96" x2="17.78" y2="43.18" width="0.1524" layer="91"/>
-<pinref part="IC2" gate="G$1" pin="R2OUT"/>
-<wire x1="17.78" y1="43.18" x2="38.1" y2="43.18" width="0.1524" layer="91"/>
-</segment>
-</net>
